File: z1-cc1120.sch (EAGLE design)
At the start: 13 parts, among them X1 PN61729-S

Commit message: added CCA_STATUS
Connections:
- new net RADIO_CCA_STATUS: U$1.TB3, U$2.GPIO3
Changed lines of the file:
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@@
+</segment>
+</net>
+<net name="RADIO_CCA_STATUS" class="0">
+<segment>
+<pinref part="U$2" gate="G$1" pin="GPIO3"/>
+<wire x1="220.98" y1="101.6" x2="251.46" y2="101.6" width="0.1524" layer="91"/>
+<label x="226.06" y="101.6" size="1.778" layer="95"/>
+</segment>
+<segment>
+<pinref part="U$1" gate="G$1" pin="TB3"/>
+<wire x1="30.48" y1="104.14" x2="5.08" y2="104.14" width="0.1524" layer="91"/>
+<label x="5.08" y="104.14" size="1.778" layer="95"/>
 </segment>
 </net>

Commit message: added !rst and cca status onto debug header
Parts:
- JP1: device pinhead:PINHD-1X6 -> pinhead:PINHD-1X8
Connections:
- net GND: now also JP1.8; no longer JP1.6
- net RADIO_!RST: now also JP1.6
- net RADIO_CCA_STATUS: now also JP1.7
Changed lines of the file:
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@@
 <part name="L1" library="resistor" deviceset="L-EU" device="L3230M" value="10mH"/>
 <part name="L2" library="resistor" deviceset="L-EU" device="L3230M" value="10mH"/>
-<part name="JP1" library="pinhead" deviceset="PINHD-1X6" device=""/>
+<part name="JP1" library="pinhead" deviceset="PINHD-1X8" device=""/>
 <part name="GND3" library="supply1" deviceset="GND" device=""/>
 <part name="R3" library="resistor" deviceset="R-EU_" device="R0805" value="1K"/>
@@
 <instance part="L1" gate="G$1" x="154.94" y="45.72" rot="R270"/>
 <instance part="L2" gate="G$1" x="154.94" y="38.1" rot="R270"/>
-<instance part="JP1" gate="A" x="172.72" y="152.4"/>
-<instance part="GND3" gate="1" x="160.02" y="144.78"/>
+<instance part="JP1" gate="A" x="172.72" y="149.86"/>
+<instance part="GND3" gate="1" x="157.48" y="139.7"/>
 <instance part="R3" gate="G$1" x="175.26" y="93.98" rot="R180"/>
 </instances>
@@
 </segment>
 <segment>
+<pinref part="JP1" gate="A" pin="8"/>
 <pinref part="GND3" gate="1" pin="GND"/>
-<pinref part="JP1" gate="A" pin="6"/>
-<wire x1="170.18" y1="147.32" x2="160.02" y2="147.32" width="0.1524" layer="91"/>
+<wire x1="170.18" y1="142.24" x2="157.48" y2="142.24" width="0.1524" layer="91"/>
 </segment>
 </net>
@@
 <segment>
 <pinref part="JP1" gate="A" pin="3"/>
-<wire x1="170.18" y1="154.94" x2="149.86" y2="154.94" width="0.1524" layer="91"/>
-<label x="149.86" y="154.94" size="1.778" layer="95"/>
+<wire x1="170.18" y1="154.94" x2="137.16" y2="154.94" width="0.1524" layer="91"/>
+<label x="137.16" y="154.94" size="1.778" layer="95"/>
 </segment>
 </net>
@@
 <segment>
 <pinref part="JP1" gate="A" pin="2"/>
-<wire x1="170.18" y1="157.48" x2="149.86" y2="157.48" width="0.1524" layer="91"/>
-<label x="149.86" y="157.48" size="1.778" layer="95"/>
+<wire x1="170.18" y1="157.48" x2="137.16" y2="157.48" width="0.1524" layer="91"/>
+<label x="137.16" y="157.48" size="1.778" layer="95"/>
 </segment>
 </net>
@@
 <segment>
 <pinref part="JP1" gate="A" pin="1"/>
-<wire x1="170.18" y1="160.02" x2="149.86" y2="160.02" width="0.1524" layer="91"/>
-<label x="149.86" y="160.02" size="1.778" layer="95"/>
+<wire x1="170.18" y1="160.02" x2="137.16" y2="160.02" width="0.1524" layer="91"/>
+<label x="137.16" y="160.02" size="1.778" layer="95"/>
 </segment>
 </net>
@@
 <segment>
 <pinref part="JP1" gate="A" pin="4"/>
-<wire x1="170.18" y1="152.4" x2="149.86" y2="152.4" width="0.1524" layer="91"/>
-<label x="149.86" y="152.4" size="1.778" layer="95"/>
+<wire x1="170.18" y1="152.4" x2="137.16" y2="152.4" width="0.1524" layer="91"/>
+<label x="137.16" y="152.4" size="1.778" layer="95"/>
 </segment>
 <segment>
@@
 <segment>
 <pinref part="JP1" gate="A" pin="5"/>
-<wire x1="170.18" y1="149.86" x2="149.86" y2="149.86" width="0.1524" layer="91"/>
-<label x="149.86" y="149.86" size="1.778" layer="95"/>
+<wire x1="170.18" y1="149.86" x2="137.16" y2="149.86" width="0.1524" layer="91"/>
+<label x="137.16" y="149.86" size="1.778" layer="95"/>
 </segment>
 <segment>
@@
 <label x="12.7" y="86.36" size="1.778" layer="95"/>
 </segment>
+<segment>
+<pinref part="JP1" gate="A" pin="6"/>
+<wire x1="170.18" y1="147.32" x2="137.16" y2="147.32" width="0.1524" layer="91"/>
+<label x="137.16" y="147.32" size="1.778" layer="95"/>
+</segment>
 </net>
 <net name="RADIO_CCA_STATUS" class="0">
@@
 <label x="5.08" y="104.14" size="1.778" layer="95"/>
 </segment>
-</net>
+<segment>
+<pinref part="JP1" gate="A" pin="7"/>
+<wire x1="170.18" y1="144.78" x2="137.16" y2="144.78" width="0.1524" layer="91"/>
+<label x="137.16" y="144.78" size="1.778" layer="95"/>
+</segment>
+</net>

Commit message: now very similar length usb tracks
Connections:
- net USB_D+ renamed USB_P
- net USB_D- renamed USB_N
Changed lines of the file:
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@@
 <class number="0" name="default" width="0" drill="0">
+</class>
+<class number="1" name="usb" width="0.3048" drill="0">
+<clearance class="1" value="0.1524"/>
 </class>
 </classes>
@@
 </segment>
 </net>
-<net name="USB_D+" class="0">
+<net name="USB_P" class="1">
 <segment>
 <pinref part="U$1" gate="G$1" pin="D_P"/>
@@
 </segment>
 </net>
-<net name="USB_D-" class="0">
+<net name="USB_N" class="1">
 <segment>
 <pinref part="U$1" gate="G$1" pin="D_N"/>
